File: pcb/wzhooh.kicad_sch (KiCad schematic)
At the start: 4 parts, among them U1 Pico, U2 DA08-11SURKWA, U3 DA08-11SURKWA, U4 DA08-11SURKWA

Commit message: pcb rev:0x01
Parts:
- added C1, C2, C3: 1nF, Capacitor_THT:C_Disc_D4.7mm_W2.5mm_P5.00mm, symbol Device:C
- added C4: 10uF, Capacitor_THT:CP_Radial_D7.5mm_P2.50mm, symbol Device:C_Polarized
- added H1, H2: MountingHole, MountingHole:MountingHole_3.2mm_M3, symbol Mechanical:MountingHole
- added J1: Sensor1, Connector_PinHeader_2.54mm:PinHeader_1x03_P2.54mm_Horizontal, symbol Connector_Generic:Conn_01x03
- added J2: Sensor2, Connector_PinHeader_2.54mm:PinHeader_1x03_P2.54mm_Horizontal, symbol Connector_Generic:Conn_01x03
- added J3: Sensor3, Connector_PinHeader_2.54mm:PinHeader_1x03_P2.54mm_Horizontal, symbol Connector_Generic:Conn_01x03
- added Q1, Q2, Q3, Q4, Q5, Q6: 2N3905, Package_TO_SOT_THT:TO-92_Inline, symbol Transistor_BJT:2N3905
- added R1, R2, R3, R4, R5, R6, R7, R8: 50Ω, Resistor_THT:R_Axial_DIN0207_L6.3mm_D2.5mm_P2.54mm_Vertical, symbol Device:R
- added R10, R13, R16: 100KΩ, Resistor_THT:R_Axial_DIN0207_L6.3mm_D2.5mm_P2.54mm_Vertical, symbol Device:R
- added R11, R12, R14, R15, R17, R18, R19, R20, R21, R22, R23, R9: 330Ω, Resistor_THT:R_Axial_DIN0207_L6.3mm_D2.5mm_P2.54mm_Vertical, symbol Device:R
- added SW1: Button1, Button_Switch_THT:SW_PUSH_6mm_H13mm, symbol Switch:SW_Push
- added SW2: Button2, Button_Switch_THT:SW_PUSH_6mm_H13mm, symbol Switch:SW_Push
- added SW3: Button3, Button_Switch_THT:SW_PUSH_6mm_H13mm, symbol Switch:SW_Push
- added U1: ULN2803A, Package_DIP:DIP-18_W7.62mm, symbol Transistor_Array:ULN2803A
- renumbered U1 to U2, U2 to U3, U3 to U4, U4 to U5
Connections:
- net SEG_A: now also R1.1
- net SEG_B: now also R2.1
- net SEG_C: now also R3.1
- net SEG_D: now also R4.1
- net SEG_DP: now also R8.1
- net SEG_E: now also R5.1
- net SEG_F: now also R6.1
- net SEG_G: now also R7.1
- net at U3.13 (DIG2_CA): now also Q4.3 (C)
- net at U3.14 (DIG1_CA): now also Q1.3 (C)
- net at U4.13 (DIG2_CA): now also Q5.3 (C)
- net at U4.14 (DIG1_CA): now also Q2.3 (C)
- net BTN_1: now reaches U2.10 (GPIO7)
- net BTN_1: now also C1.1, SW1.2
- net at U2.11 (GPIO8): now also U1.1 (I1)
- net at U2.12 (GPIO9): now also U1.2 (I2)
- net GND: now reaches U2.13 (GND)
- net GND: now also U2.18 (GND), U2.23 (GND), U2.28 (GND), U2.3 (GND), U2.38 (GND), U2.42 (GND), U2.8 (GND), C1.2, C2.2, C3.2, C4.2, J1.1 (Pin_1), J2.1 (Pin_1), J3.1 (Pin_1), SW1.1, SW2.1, SW3.1, U1.9 (GND)
- net at U2.14 (GPIO10): now also U1.3 (I3)
- net at U2.15 (GPIO11): now also U1.4 (I4)
- net at U2.16 (GPIO12): now also U1.5 (I5)
- net at U2.17 (GPIO13): now also U1.6 (I6)
- net at U2.19 (GPIO14): now also U1.7 (I7)
- net at U2.20 (GPIO15): now also U1.8 (I8)
- net COM_6: now reaches U2.21 (GPIO16)
- net COM_6: now also R23.2
- net COM_5: now reaches U2.22 (GPIO17)
- net COM_5: now also R20.2
- net COM_4: now reaches U2.24 (GPIO18)
- net COM_4: now also R22.2
- net COM_3: now reaches U2.25 (GPIO19)
- net COM_3: now also R19.2
- net COM_2: now reaches U2.26 (GPIO20)
- net COM_2: now also R21.2
- net COM_1: now reaches U2.27 (GPIO21)
- net COM_1: now also R18.2
- net SENSE_3: now reaches U2.31 (GPIO26_ADC0)
- net SENSE_3: now also R17.2
- net SENSE_2: now reaches U2.32 (GPIO27_ADC1)
- net SENSE_2: now also R14.2
- net SENSE_1: now reaches U2.34 (GPIO28_ADC2)
- net SENSE_1: now also R11.2
- net VDD: now reaches U2.36 (3V3)
- net VDD: now also C4.1, Q1.1 (E), Q2.1 (E), Q3.1 (E), Q4.1 (E), Q5.1 (E), Q6.1 (E), R10.2, R12.2, R13.2, R15.2, R16.2, R9.2, U1.10 (COM)
- net BTN_3: now reaches U2.7 (GPIO5)
- net BTN_3: now also C3.1, SW3.2
- net BTN_2: now reaches U2.9 (GPIO6)
- net BTN_2: now also C2.1, SW2.2
- net at U5.13 (DIG2_CA): now also Q6.3 (C)
- net at U5.14 (DIG1_CA): now also Q3.3 (C)
- new net: Q5.2 (B), R22.1
- new net: Q2.2 (B), R19.1
- new net: J1.2 (Pin_2), R10.1, R11.1
- new net: R2.2, U1.17 (O2)
- new net: Q3.2 (B), R20.1
- new net: R8.2, U1.11 (O8)
- new net: R7.2, U1.12 (O7)
- new net: R6.2, U1.13 (O6)
- new net: R5.2, U1.14 (O5)
- new net: R4.2, U1.15 (O4)
- new net: R3.2, U1.16 (O3)
- new net: R1.2, U1.18 (O1)
- new net: Q6.2 (B), R23.1
- new net: J1.3 (Pin_3), R9.1
- new net: Q1.2 (B), R18.1
- new net: J2.2 (Pin_2), R13.1, R14.1
- new net: J2.3 (Pin_3), R12.1
- new net: Q4.2 (B), R21.1
- new net: J3.2 (Pin_2), R16.1, R17.1
- new net: J3.3 (Pin_3), R15.1
- no-connect marks 0 -> 14
Other:
- company: (none) -> vitaly.codes
- title: (none) -> Wzhooh
- moved on the sheet: U2, U3, U4, U5

Commit message: add BOM
Parts:
- Q1, Q2, Q3, Q4, Q5: value 2N3905 -> 2N2907
- Q6: value 2N3905 -> 2N2907; footprint Package_TO_SOT_THT:TO-92_Inline -> https://www.mouser.com/datasheet/2/849/2n2907a-2577411.pdf
Changed lines of the file:
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@@
       (effects (font (size 1.27 1.27)))
     )
-    (property "Value" "2N3905" (at 254 92.71 90)
+    (property "Value" "2N2907" (at 254 92.71 90)
       (effects (font (size 1.27 1.27)))
     )
@@
       (effects (font (size 1.27 1.27) italic) (justify left) hide)
     )
-    (property "Datasheet" "https://www.nteinc.com/specs/original/2N3905_06.pdf" (at 254 99.06 0)
+    (property "Datasheet" "https://www.mouser.com/datasheet/2/849/2n2907a-2577411.pdf" (at 254 99.06 0)
       (effects (font (size 1.27 1.27)) (justify left) hide)
     )
@@
       (effects (font (size 1.27 1.27)))
     )
-    (property "Value" "2N3905" (at 187.96 143.51 90)
+    (property "Value" "2N2907" (at 187.96 143.51 90)
       (effects (font (size 1.27 1.27)))
     )
@@
       (effects (font (size 1.27 1.27) italic) (justify left) hide)
     )
-    (property "Datasheet" "https://www.nteinc.com/specs/original/2N3905_06.pdf" (at 187.96 149.86 0)
+    (property "Datasheet" "https://www.mouser.com/datasheet/2/849/2n2907a-2577411.pdf" (at 187.96 149.86 0)
       (effects (font (size 1.27 1.27)) (justify left) hide)
     )
@@
       (effects (font (size 1.27 1.27)))
     )
-    (property "Value" "2N3905" (at 187.96 92.71 90)
+    (property "Value" "2N2907" (at 187.96 92.71 90)
       (effects (font (size 1.27 1.27)))
     )
@@
       (effects (font (size 1.27 1.27) italic) (justify left) hide)
     )
-    (property "Datasheet" "https://www.nteinc.com/specs/original/2N3905_06.pdf" (at 187.96 99.06 0)
+    (property "Datasheet" "https://www.mouser.com/datasheet/2/849/2n2907a-2577411.pdf" (at 187.96 99.06 0)
       (effects (font (size 1.27 1.27)) (justify left) hide)
     )
@@
       (effects (font (size 1.27 1.27)))
     )
-    (property "Value" "2N3905" (at 187.96 41.91 90)
+    (property "Value" "2N2907" (at 187.96 41.91 90)
       (effects (font (size 1.27 1.27)))
     )
@@
       (effects (font (size 1.27 1.27) italic) (justify left) hide)
     )
-    (property "Datasheet" "https://www.nteinc.com/specs/original/2N3905_06.pdf" (at 187.96 48.26 0)
+    (property "Datasheet" "https://www.mouser.com/datasheet/2/849/2n2907a-2577411.pdf" (at 187.96 48.26 0)
       (effects (font (size 1.27 1.27)) (justify left) hide)
     )
@@
       (effects (font (size 1.27 1.27)))
     )
-    (property "Value" "2N3905" (at 254 143.51 90)
-      (effects (font (size 1.27 1.27)))
-    )
-    (property "Footprint" "Package_TO_SOT_THT:TO-92_Inline" (at 255.905 144.78 0)
+    (property "Value" "2N2907" (at 254 143.51 90)
+      (effects (font (size 1.27 1.27)))
+    )
+    (property "Footprint" "https://www.mouser.com/datasheet/2/849/2n2907a-2577411.pdf" (at 255.905 144.78 0)
       (effects (font (size 1.27 1.27) italic) (justify left) hide)
     )
@@
       (effects (font (size 1.27 1.27)))
     )
-    (property "Value" "2N3905" (at 254 41.91 90)
+    (property "Value" "2N2907" (at 254 41.91 90)
       (effects (font (size 1.27 1.27)))
     )
@@
       (effects (font (size 1.27 1.27) italic) (justify left) hide)
     )
-    (property "Datasheet" "https://www.nteinc.com/specs/original/2N3905_06.pdf" (at 254 48.26 0)
+    (property "Datasheet" "https://www.mouser.com/datasheet/2/849/2n2907a-2577411.pdf" (at 254 48.26 0)
       (effects (font (size 1.27 1.27)) (justify left) hide)
     )

Commit message: rev: 0x01
Parts:
- R1, R2, R3, R4, R5, R6, R7, R8: value 50Ω -> 33Ω
Changed lines of the file:
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@@
       (effects (font (size 1.27 1.27)))
     )
-    (property "Value" "50Ω" (at 34.29 62.23 90)
+    (property "Value" "33Ω" (at 34.29 62.23 90)
       (effects (font (size 1.27 1.27)))
     )
@@
       (effects (font (size 1.27 1.27)))
     )
-    (property "Value" "50Ω" (at 34.29 57.15 90)
+    (property "Value" "33Ω" (at 34.29 57.15 90)
       (effects (font (size 1.27 1.27)))
     )
@@
       (effects (font (size 1.27 1.27)))
     )
-    (property "Value" "50Ω" (at 34.29 67.31 90)
+    (property "Value" "33Ω" (at 34.29 67.31 90)
       (effects (font (size 1.27 1.27)))
     )
@@
       (effects (font (size 1.27 1.27)))
     )
-    (property "Value" "50Ω" (at 34.29 77.47 90)
+    (property "Value" "33Ω" (at 34.29 77.47 90)
       (effects (font (size 1.27 1.27)))
     )
@@
       (effects (font (size 1.27 1.27)))
     )
-    (property "Value" "50Ω" (at 34.29 72.39 90)
+    (property "Value" "33Ω" (at 34.29 72.39 90)
       (effects (font (size 1.27 1.27)))
     )
@@
       (effects (font (size 1.27 1.27)))
     )
-    (property "Value" "50Ω" (at 34.29 82.55 90)
+    (property "Value" "33Ω" (at 34.29 82.55 90)
       (effects (font (size 1.27 1.27)))
     )
@@
       (effects (font (size 1.27 1.27)))
     )
-    (property "Value" "50Ω" (at 34.29 87.63 90)
+    (property "Value" "33Ω" (at 34.29 87.63 90)
       (effects (font (size 1.27 1.27)))
     )
@@
       (effects (font (size 1.27 1.27)))
     )
-    (property "Value" "50Ω" (at 34.29 92.71 90)
-      (effects (font (size 1.27 1.27)))
-    )
+    (property "Value" "33Ω" (at 34.29 92.71 90)
+      (effects (font (size 1.27 1.27)))
+    )
